File: clocks.sch (KiCad schematic (older format))
At the start: 10 parts, among them J2 UPDI TTL, U10 74HC3G34DP,125, U2 Si5351A-B-GT, U5 ATtiny1614-SS, Y1 25MHZ 8PF

Commit message: added 3V3 section for clock generator
Parts:
- added C3: 10uF, Capacitor_SMD:C_0805_2012Metric_Pad1.15x1.40mm_HandSolder, symbol Device:C_Small
- added C4: 22uF, Capacitor_SMD:C_0805_2012Metric_Pad1.15x1.40mm_HandSolder, symbol Device:C_Small
- added U11: AZ1117CH-3.3TRG1, Package_TO_SOT_SMD:SOT-223-3_TabPin2, symbol Regulator_Linear:AZ1117-3.3
Connections:
- net labels added: CLK_10_Mhz
- net labels removed: CLK_7_3728_Mhz
- wire segments 29 -> 41
Changed lines of the file:
@@
 $Descr A4 11693 8268
 encoding utf-8
-Sheet 3 3
+Sheet 2 2
 Title ""
 Date ""
@@
 CLK_100Mhz
 Text HLabel 8030 2280 2    50   Output ~ 0
-CLK_7_3728_Mhz
+CLK_10_Mhz
 Text HLabel 8030 2480 2    50   Output ~ 0
 CLK_1Mhz
@@
 Text GLabel 8915 805  1    50   Output ~ 0
 5V
+$Comp
+L Regulator_Linear:AZ1117-3.3 U11
+U 1 1 5D14EF24
+P 2615 1005
+F 0 "U11" H 2615 1247 50  0000 C CNN
+F 1 "AZ1117CH-3.3TRG1" H 2615 1156 50  0000 C CNN
+F 2 "Package_TO_SOT_SMD:SOT-223-3_TabPin2" H 2615 1255 50  0001 C CIN
+F 3 "https://www.mouser.com/datasheet/2/115/AZ1117C-1147948.pdf" H 2615 1005 50  0001 C CNN
+	1    2615 1005
+	1    0    0    -1
+$EndComp
+$Comp
+L Device:C_Small C3
+U 1 1 5D1521F5
+P 2000 1100
+F 0 "C3" H 2092 1146 50  0000 L CNN
+F 1 "10uF" H 2092 1055 50  0000 L CNN
+F 2 "Capacitor_SMD:C_0805_2012Metric_Pad1.15x1.40mm_HandSolder" H 2000 1100 50  0001 C CNN
+F 3 "https://www.mouser.com/datasheet/2/396/mlcc02_e-1307760.pdf" H 2000 1100 50  0001 C CNN
+F 4 "Multilayer Ceramic Capacitors MLCC - SMD/SMT 0805 6.3V 10uF 10% X7R" H 2092 1246 50  0001 C CNN "Description"
+F 5 "Taiyo Yuden" H 2000 1100 50  0001 C CNN "MFR"
+F 6 "JMK107B7474KA-T" H 2000 1100 50  0001 C CNN "MPN"
+F 7 "963-JMK107B7474KA-T" H 2092 1246 50  0001 C CNN "SPN"
+F 8 "Mouser" H 2000 1100 50  0001 C CNN "SPR"
+F 9 "https://www.mouser.com/ProductDetail/963-JMK107B7474KA-T" H 2092 1246 50  0001 C CNN "SPURL"
+	1    2000 1100
+	1    0    0    -1
+$EndComp
+$Comp
+L Device:C_Small C4
+U 1 1 5D152201
+P 3105 1100
+F 0 "C4" H 3197 1146 50  0000 L CNN
+F 1 "22uF" H 3197 1055 50  0000 L CNN
+F 2 "Capacitor_SMD:C_0805_2012Metric_Pad1.15x1.40mm_HandSolder" H 3105 1100 50  0001 C CNN
+F 3 "https://www.mouser.com/datasheet/2/396/mlcc02_e-1307760.pdf" H 3105 1100 50  0001 C CNN
+F 4 "Multilayer Ceramic Capacitors MLCC - SMD/SMT 0603 6.3V 0.47uF 10% X7R" H 3197 1246 50  0001 C CNN "Description"
+F 5 "Taiyo Yuden" H 3105 1100 50  0001 C CNN "MFR"
+F 6 "JMK107B7474KA-T" H 3105 1100 50  0001 C CNN "MPN"
+F 7 "963-JMK107B7474KA-T" H 3197 1246 50  0001 C CNN "SPN"
+F 8 "Mouser" H 3105 1100 50  0001 C CNN "SPR"
+F 9 "https://www.mouser.com/ProductDetail/963-JMK107B7474KA-T" H 3197 1246 50  0001 C CNN "SPURL"
+	1    3105 1100
+	1    0    0    -1
+$EndComp
+Wire Wire Line
+	2000 1200 2000 1385
+Wire Wire Line
+	3105 1385 3105 1200
+Wire Wire Line
+	2000 1385 2615 1385
+Wire Wire Line
+	2615 1305 2615 1385
+Connection ~ 2615 1385
+Wire Wire Line
+	2615 1385 3105 1385
+Wire Wire Line
+	2615 1385 2615 1475
+$Comp
+L power:GND #PWR?
+U 1 1 5D15A1D6
+P 2615 1475
+AR Path="/5D15A1D6" Ref="#PWR?"  Part="1"
+AR Path="/5D0F9837/5D15A1D6" Ref="#PWR?"  Part="1"
+AR Path="/5CFABACD/5D15A1D6" Ref="#PWR?"  Part="1"
+AR Path="/5CFABACD/5CFFC458/5D15A1D6" Ref="#PWR?"  Part="1"
+AR Path="/5D65A6A0/5D15A1D6" Ref="#PWR08"  Part="1"
+F 0 "#PWR08" H 2615 1225 50  0001 C CNN
+F 1 "GND" H 2620 1302 50  0000 C CNN
+F 2 "" H 2615 1475 50  0001 C CNN
+F 3 "" H 2615 1475 50  0001 C CNN
+	1    2615 1475
+	-1   0    0    -1
+$EndComp
+Wire Wire Line
+	2915 1005 3105 1005
+Wire Wire Line
+	3105 1005 3105 1000
+Wire Wire Line
+	3105 1005 3410 1005
+Connection ~ 3105 1005
+Wire Wire Line
+	1780 1000 2000 1000
+Wire Wire Line
+	2315 1000 2315 1005
+Connection ~ 2000 1000
+Wire Wire Line
+	2000 1000 2315 1000
+Text GLabel 3410 1005 2    50   Output ~ 0
+3V3
+Text GLabel 1780 1000 0    50   Input ~ 0
+5V
 $EndSCHEMATC

Commit message: larger sheet, connected more pins
Parts:
- added C15, C16: 100nF, Capacitor_SMD:C_0805_2012Metric_Pad1.15x1.40mm_HandSolder, symbol Device:C_Small
- U10: symbol 74xx:74HC3G34DP,125 -> sbc_z80-rescue:74HC3G34DP,125-74xx
Connections:
- net labels added: +3V3, +5V
- net labels removed: 3V3, 5V
- wire segments 41 -> 50
Other:
- moved on the sheet: C1, C2, C3, C4, J2, R1, R2, R3, U2, U5, Y1

Commit message: reordered resistors
Parts:
- removed U11: AZ1117CH-3.3TRG1, Package_TO_SOT_SMD:SOT-223-3_TabPin2, symbol Regulator_Linear:AZ1117-3.3
- added U11: MIC5356-SGYMME, Package_SO:MSOP-8-1EP_3x3mm_P0.65mm_EP2.5x3mm_Mask1.73x2.36mm_ThermalVias, symbol Regulator_Linear:MIC5356-SGYMME
- J2: footprint Connector_PinHeader_2.54mm:PinHeader_1x03_P2.54mm_Vertical -> Connector_PinHeader_1.27mm:PinHeader_1x03_P1.27mm_Vertical
Connections:
- net labels added: CLK_7_3728_Mhz
- net labels removed: CLK_1Mhz
- wire segments 50 -> 53
- no-connect marks 9 -> 10
Other:
- moved on the sheet: C3, C4
Changed lines of the file:
@@
 F 0 "J2" H 3335 4130 50  0000 C CNN
 F 1 "UPDI TTL" H 3340 4000 50  0000 C CNN
-F 2 "Connector_PinHeader_2.54mm:PinHeader_1x03_P2.54mm_Vertical" H 3340 3725 50  0001 C CNN
+F 2 "Connector_PinHeader_1.27mm:PinHeader_1x03_P1.27mm_Vertical" H 3340 3725 50  0001 C CNN
 F 3 "~" H 3340 3725 50  0001 C CNN
 	1    3340 3725
@@
 CLK_10_Mhz
 Text HLabel 8605 3725 2    50   Output ~ 0
-CLK_1Mhz
+CLK_7_3728_Mhz
 $Comp
 L sbc_z80-rescue:74HC3G34DP,125-74xx U10
@@
 L Device:C_Small C3
 U 1 1 5D1521F5
-P 3810 1760
-F 0 "C3" H 3902 1806 50  0000 L CNN
-F 1 "10uF" H 3902 1715 50  0000 L CNN
-F 2 "Capacitor_SMD:C_0805_2012Metric_Pad1.15x1.40mm_HandSolder" H 3810 1760 50  0001 C CNN
-F 3 "https://www.mouser.com/datasheet/2/396/mlcc02_e-1307760.pdf" H 3810 1760 50  0001 C CNN
-F 4 "Multilayer Ceramic Capacitors MLCC - SMD/SMT 0805 6.3V 10uF 10% X7R" H 3902 1906 50  0001 C CNN "Description"
-F 5 "Taiyo Yuden" H 3810 1760 50  0001 C CNN "MFR"
-F 6 "JMK107B7474KA-T" H 3810 1760 50  0001 C CNN "MPN"
-F 7 "963-JMK107B7474KA-T" H 3902 1906 50  0001 C CNN "SPN"
-F 8 "Mouser" H 3810 1760 50  0001 C CNN "SPR"
-F 9 "https://www.mouser.com/ProductDetail/963-JMK107B7474KA-T" H 3902 1906 50  0001 C CNN "SPURL"
-	1    3810 1760
+P 3695 2060
+F 0 "C3" H 3787 2106 50  0000 L CNN
+F 1 "10uF" H 3787 2015 50  0000 L CNN
+F 2 "Capacitor_SMD:C_0805_2012Metric_Pad1.15x1.40mm_HandSolder" H 3695 2060 50  0001 C CNN
+F 3 "https://www.mouser.com/datasheet/2/396/mlcc02_e-1307760.pdf" H 3695 2060 50  0001 C CNN
+F 4 "Multilayer Ceramic Capacitors MLCC - SMD/SMT 0805 6.3V 10uF 10% X7R" H 3787 2206 50  0001 C CNN "Description"
+F 5 "Taiyo Yuden" H 3695 2060 50  0001 C CNN "MFR"
+F 6 "JMK107B7474KA-T" H 3695 2060 50  0001 C CNN "MPN"
+F 7 "963-JMK107B7474KA-T" H 3787 2206 50  0001 C CNN "SPN"
+F 8 "Mouser" H 3695 2060 50  0001 C CNN "SPR"
+F 9 "https://www.mouser.com/ProductDetail/963-JMK107B7474KA-T" H 3787 2206 50  0001 C CNN "SPURL"
+	1    3695 2060
 	1    0    0    -1
 $EndComp
@@
 L Device:C_Small C4
 U 1 1 5D152201
-P 4915 1755
-F 0 "C4" H 5007 1801 50  0000 L CNN
-F 1 "22uF" H 5007 1710 50  0000 L CNN
-F 2 "Capacitor_SMD:C_0805_2012Metric_Pad1.15x1.40mm_HandSolder" H 4915 1755 50  0001 C CNN
-F 3 "https://www.mouser.com/datasheet/2/396/mlcc02_e-1307760.pdf" H 4915 1755 50  0001 C CNN
-F 4 "Multilayer Ceramic Capacitors MLCC - SMD/SMT 0603 6.3V 0.47uF 10% X7R" H 5007 1901 50  0001 C CNN "Description"
-F 5 "Taiyo Yuden" H 4915 1755 50  0001 C CNN "MFR"
-F 6 "JMK107B7474KA-T" H 4915 1755 50  0001 C CNN "MPN"
-F 7 "963-JMK107B7474KA-T" H 5007 1901 50  0001 C CNN "SPN"
-F 8 "Mouser" H 4915 1755 50  0001 C CNN "SPR"
-F 9 "https://www.mouser.com/ProductDetail/963-JMK107B7474KA-T" H 5007 1901 50  0001 C CNN "SPURL"
-	1    4915 1755
-	1    0    0    -1
-$EndComp
-Wire Wire Line
-	4915 2040 4915 1855
-Wire Wire Line
-	3810 2040 4425 2040
-Wire Wire Line
-	4425 1960 4425 2040
-Connection ~ 4425 2040
-Wire Wire Line
-	4425 2040 4915 2040
-Wire Wire Line
-	4425 2040 4425 2130
+P 5000 2155
+F 0 "C4" H 5092 2201 50  0000 L CNN
+F 1 "22uF" H 5092 2110 50  0000 L CNN
+F 2 "Capacitor_SMD:C_0805_2012Metric_Pad1.15x1.40mm_HandSolder" H 5000 2155 50  0001 C CNN
+F 3 "https://www.mouser.com/datasheet/2/396/mlcc02_e-1307760.pdf" H 5000 2155 50  0001 C CNN
+F 4 "Multilayer Ceramic Capacitors MLCC - SMD/SMT 0603 6.3V 0.47uF 10% X7R" H 5092 2301 50  0001 C CNN "Description"
+F 5 "Taiyo Yuden" H 5000 2155 50  0001 C CNN "MFR"
+F 6 "JMK107B7474KA-T" H 5000 2155 50  0001 C CNN "MPN"
+F 7 "963-JMK107B7474KA-T" H 5092 2301 50  0001 C CNN "SPN"
+F 8 "Mouser" H 5000 2155 50  0001 C CNN "SPR"
+F 9 "https://www.mouser.com/ProductDetail/963-JMK107B7474KA-T" H 5092 2301 50  0001 C CNN "SPURL"
+	1    5000 2155
+	1    0    0    -1
+$EndComp
+Wire Wire Line
+	4410 2360 4410 2405
 $Comp
 L power:GND #PWR?
 U 1 1 5D15A1D6
-P 4425 2130
+P 4410 2450
 AR Path="/5D15A1D6" Ref="#PWR?"  Part="1"
 AR Path="/5D0F9837/5D15A1D6" Ref="#PWR?"  Part="1"
@@
 AR Path="/5CFABACD/5CFFC458/5D15A1D6" Ref="#PWR?"  Part="1"
 AR Path="/5D65A6A0/5D15A1D6" Ref="#PWR08"  Part="1"
-F 0 "#PWR08" H 4425 1880 50  0001 C CNN
-F 1 "GND" H 4430 1957 50  0000 C CNN
-F 2 "" H 4425 2130 50  0001 C CNN
-F 3 "" H 4425 2130 50  0001 C CNN
-	1    4425 2130
+F 0 "#PWR08" H 4410 2200 50  0001 C CNN
+F 1 "GND" H 4415 2277 50  0000 C CNN
+F 2 "" H 4410 2450 50  0001 C CNN
+F 3 "" H 4410 2450 50  0001 C CNN
+	1    4410 2450
 	-1   0    0    -1
 $EndComp
 Wire Wire Line
-	4725 1660 4915 1660
-Wire Wire Line
-	4915 1660 4915 1655
-Wire Wire Line
-	4915 1660 5130 1660
-Connection ~ 4915 1660
-$Comp
-L Regulator_Linear:AZ1117-3.3 U11
-U 1 1 5D14EF24
-P 4425 1660
-F 0 "U11" H 4425 1902 50  0000 C CNN
-F 1 "AZ1117CH-3.3TRG1" H 4425 1811 50  0000 C CNN
-F 2 "Package_TO_SOT_SMD:SOT-223-3_TabPin2" H 4425 1910 50  0001 C CIN
-F 3 "https://www.mouser.com/datasheet/2/115/AZ1117C-1147948.pdf" H 4425 1660 50  0001 C CNN
-	1    4425 1660
-	1    0    0    -1
-$EndComp
-Wire Wire Line
-	4125 1660 3810 1660
-Connection ~ 3810 1660
-Wire Wire Line
-	3810 1860 3810 2040
+	4810 2060 5000 2060
+Wire Wire Line
+	5000 2060 5000 2055
+Wire Wire Line
+	5000 2060 5215 2060
+Connection ~ 5000 2060
+Connection ~ 3695 1960
 $Comp
 L power:+3V3 #PWR0113
 U 1 1 5EFB1AF8
-P 5220 1660
-F 0 "#PWR0113" H 5220 1510 50  0001 C CNN
-F 1 "+3V3" V 5235 1788 50  0000 L CNN
-F 2 "" H 5220 1660 50  0001 C CNN
-F 3 "" H 5220 1660 50  0001 C CNN
-	1    5220 1660
+P 5305 2060
+F 0 "#PWR0113" H 5305 1910 50  0001 C CNN
+F 1 "+3V3" V 5320 2188 50  0000 L CNN
+F 2 "" H 5305 2060 50  0001 C CNN
+F 3 "" H 5305 2060 50  0001 C CNN
+	1    5305 2060
 	0    1    1    0
 $EndComp
@@
 L power:PWR_FLAG #FLG0101
 U 1 1 5EFC0EF3
-P 5130 1660
-F 0 "#FLG0101" H 5130 1735 50  0001 C CNN
-F 1 "PWR_FLAG" H 5130 1833 50  0000 C CNN
-F 2 "" H 5130 1660 50  0001 C CNN
-F 3 "~" H 5130 1660 50  0001 C CNN
-	1    5130 1660
-	1    0    0    -1
-$EndComp
-Connection ~ 5130 1660
-Wire Wire Line
-	5130 1660 5220 1660
+P 5215 2060
+F 0 "#FLG0101" H 5215 2135 50  0001 C CNN
+F 1 "PWR_FLAG" H 5215 2233 50  0000 C CNN
+F 2 "" H 5215 2060 50  0001 C CNN
+F 3 "~" H 5215 2060 50  0001 C CNN
+	1    5215 2060
+	1    0    0    -1
+$EndComp
+Connection ~ 5215 2060
+Wire Wire Line
+	5215 2060 5305 2060
 $Comp
 L power:PWR_FLAG #FLG0102
 U 1 1 5EFC1C86
-P 3660 1660
-F 0 "#FLG0102" H 3660 1735 50  0001 C CNN
-F 1 "PWR_FLAG" H 3660 1833 50  0000 C CNN
-F 2 "" H 3660 1660 50  0001 C CNN
-F 3 "~" H 3660 1660 50  0001 C CNN
-	1    3660 1660
-	1    0    0    -1
-$EndComp
-Connection ~ 3660 1660
-Wire Wire Line
-	3660 1660 3810 1660
+P 3545 1960
+F 0 "#FLG0102" H 3545 2035 50  0001 C CNN
+F 1 "PWR_FLAG" H 3545 2133 50  0000 C CNN
+F 2 "" H 3545 1960 50  0001 C CNN
+F 3 "~" H 3545 1960 50  0001 C CNN
+	1    3545 1960
+	1    0    0    -1
+$EndComp
+Connection ~ 3545 1960
+Wire Wire Line
+	3545 1960 3695 1960
 $Comp
 L Device:C_Small C15
@@
 L power:+5V #PWR016
 U 1 1 5F57C70A
-P 3255 1660
-F 0 "#PWR016" H 3255 1510 50  0001 C CNN
-F 1 "+5V" H 3270 1833 50  0000 C CNN
-F 2 "" H 3255 1660 50  0001 C CNN
-F 3 "" H 3255 1660 50  0001 C CNN
-	1    3255 1660
-	1    0    0    -1
-$EndComp
-Wire Wire Line
-	3255 1660 3660 1660
+P 3140 1960
+F 0 "#PWR016" H 3140 1810 50  0001 C CNN
+F 1 "+5V" H 3155 2133 50  0000 C CNN
+F 2 "" H 3140 1960 50  0001 C CNN
+F 3 "" H 3140 1960 50  0001 C CNN
+	1    3140 1960
+	1    0    0    -1
+$EndComp
+Wire Wire Line
+	3140 1960 3545 1960
+$Comp
+L Regulator_Linear:MIC5356-SGYMME U11
+U 1 1 5E75D8A8
+P 4410 2060
+F 0 "U11" H 4410 2441 50  0000 C CNN
+F 1 "MIC5356-SGYMME" H 4410 2350 50  0000 C CNN
+F 2 "Package_SO:MSOP-8-1EP_3x3mm_P0.65mm_EP2.5x3mm_Mask1.73x2.36mm_ThermalVias" H 5810 1810 50  0001 C CNN
+F 3 "http://ww1.microchip.com/downloads/en/DeviceDoc/mic5355_6.pdf" H 4410 2410 50  0001 C CNN
+	1    4410 2060
+	1    0    0    -1
+$EndComp
+NoConn ~ 4810 2160
+Wire Wire Line
+	4010 2160 4010 2405
+Wire Wire Line
+	4010 2405 4410 2405
+Connection ~ 4410 2405
+Wire Wire Line
+	4410 2405 4410 2450
+Wire Wire Line
+	4010 1960 3905 1960
+Wire Wire Line
+	4010 2060 3905 2060
+Wire Wire Line
+	3905 2060 3905 1960
+Connection ~ 3905 1960
+Wire Wire Line
+	3905 1960 3695 1960
+$Comp
+L power:GND #PWR?
+U 1 1 5E77B1C8
+P 5000 2300
+AR Path="/5E77B1C8" Ref="#PWR?"  Part="1"
+AR Path="/5D0F9837/5E77B1C8" Ref="#PWR?"  Part="1"
+AR Path="/5CFABACD/5E77B1C8" Ref="#PWR?"  Part="1"
+AR Path="/5CFABACD/5CFFC458/5E77B1C8" Ref="#PWR?"  Part="1"
+AR Path="/5D65A6A0/5E77B1C8" Ref="#PWR033"  Part="1"
+F 0 "#PWR033" H 5000 2050 50  0001 C CNN
+F 1 "GND" H 5005 2127 50  0000 C CNN
+F 2 "" H 5000 2300 50  0001 C CNN
+F 3 "" H 5000 2300 50  0001 C CNN
+	1    5000 2300
+	-1   0    0    -1
+$EndComp
+Wire Wire Line
+	5000 2255 5000 2300
+$Comp
+L power:GND #PWR?
+U 1 1 5E77C6D4
+P 3695 2205
+AR Path="/5E77C6D4" Ref="#PWR?"  Part="1"
+AR Path="/5D0F9837/5E77C6D4" Ref="#PWR?"  Part="1"
+AR Path="/5CFABACD/5E77C6D4" Ref="#PWR?"  Part="1"
+AR Path="/5CFABACD/5CFFC458/5E77C6D4" Ref="#PWR?"  Part="1"
+AR Path="/5D65A6A0/5E77C6D4" Ref="#PWR032"  Part="1"
+F 0 "#PWR032" H 3695 1955 50  0001 C CNN
+F 1 "GND" H 3700 2032 50  0000 C CNN
+F 2 "" H 3695 2205 50  0001 C CNN
+F 3 "" H 3695 2205 50  0001 C CNN
+	1    3695 2205
+	-1   0    0    -1
+$EndComp
+Wire Wire Line
+	3695 2160 3695 2205
 $EndSCHEMATC

Commit message: changed part layouts
Parts:
- removed U10: 74HC3G34DP,125, Package_SO:VSSOP-8_2.4x2.1mm_P0.5mm, symbol sbc_z80-rescue:74HC3G34DP,125-74xx
- added U10: 74HC3G04DP,125, Package_SO:TSSOP-8_3x3mm_P0.65mm, symbol 74xx:74HC3G04DP,125
Other:
- moved on the sheet: C15, C16
Changed lines of the file:
@@
 CLK_7_3728_Mhz
-$Comp
-L sbc_z80-rescue:74HC3G34DP,125-74xx U10
-U 1 1 5D4A9349
-P 8305 3325
-AR Path="/5D4A9349" Ref="U10"  Part="1"
-AR Path="/5D65A6A0/5D4A9349" Ref="U10"  Part="1"
-F 0 "U10" H 8815 3635 50  0000 C CNN
-F 1 "74HC3G34DP,125" H 9265 3460 50  0000 C CNN
-F 2 "Package_SO:VSSOP-8_2.4x2.1mm_P0.5mm" H 8305 3625 50  0001 C CNN
-F 3 "http://www.ti.com/lit/gpn/sn74LS04" H 8305 3375 50  0001 C CNN
-	1    8305 3325
-	1    0    0    -1
-$EndComp
-$Comp
-L sbc_z80-rescue:74HC3G34DP,125-74xx U10
-U 2 1 5D4A9C82
-P 8305 3525
-AR Path="/5D4A9C82" Ref="U10"  Part="2"
-AR Path="/5D65A6A0/5D4A9C82" Ref="U10"  Part="2"
-F 0 "U10" H 8815 3945 50  0000 C CNN
-F 1 "74HC3G34DP,125" H 9270 4035 50  0000 C CNN
-F 2 "Package_SO:VSSOP-8_2.4x2.1mm_P0.5mm" H 8305 3825 50  0001 C CNN
-F 3 "http://www.ti.com/lit/gpn/sn74LS04" H 8305 3575 50  0001 C CNN
-	2    8305 3525
-	1    0    0    -1
-$EndComp
-$Comp
-L sbc_z80-rescue:74HC3G34DP,125-74xx U10
-U 3 1 5D4AA51A
-P 8305 3725
-AR Path="/5D4AA51A" Ref="U10"  Part="3"
-AR Path="/5D65A6A0/5D4AA51A" Ref="U10"  Part="3"
-F 0 "U10" H 8820 4260 50  0000 C CNN
-F 1 "74HC3G34DP,125" H 9255 4345 50  0000 C CNN
-F 2 "Package_SO:VSSOP-8_2.4x2.1mm_P0.5mm" H 8305 4025 50  0001 C CNN
-F 3 "http://www.ti.com/lit/gpn/sn74LS04" H 8305 3775 50  0001 C CNN
-	3    8305 3725
-	1    0    0    -1
-$EndComp
-$Comp
-L sbc_z80-rescue:74HC3G34DP,125-74xx U10
-U 4 1 5D4AAA2C
-P 9490 2350
-AR Path="/5D4AAA2C" Ref="U10"  Part="4"
-AR Path="/5D65A6A0/5D4AAA2C" Ref="U10"  Part="4"
-F 0 "U10" H 9568 2371 50  0000 L CNN
-F 1 "74HC3G34DP,125" H 9568 2280 50  0000 L CNN
-F 2 "Package_SO:VSSOP-8_2.4x2.1mm_P0.5mm" H 9490 2650 50  0001 C CNN
-F 3 "http://www.ti.com/lit/gpn/sn74LS04" H 9490 2400 50  0001 C CNN
-	4    9490 2350
-	1    0    0    -1
-$EndComp
 $Comp
 L power:GND #PWR?
@@
 L Device:C_Small C15
 U 1 1 5F1175E3
-P 2770 5580
-F 0 "C15" H 2862 5626 50  0000 L CNN
-F 1 "100nF" H 2862 5535 50  0000 L CNN
-F 2 "Capacitor_SMD:C_0805_2012Metric_Pad1.15x1.40mm_HandSolder" H 2770 5580 50  0001 C CNN
-F 3 "https://www.mouser.com/datasheet/2/396/mlcc02_e-1307760.pdf" H 2770 5580 50  0001 C CNN
-F 4 "Multilayer Ceramic Capacitors MLCC - SMD/SMT 0603 6.3V 0.47uF 10% X7R" H 2862 5726 50  0001 C CNN "Description"
-F 5 "Taiyo Yuden" H 2770 5580 50  0001 C CNN "MFR"
-F 6 "JMK107B7474KA-T" H 2770 5580 50  0001 C CNN "MPN"
-F 7 "963-JMK107B7474KA-T" H 2862 5726 50  0001 C CNN "SPN"
-F 8 "Mouser" H 2770 5580 50  0001 C CNN "SPR"
-F 9 "https://www.mouser.com/ProductDetail/963-JMK107B7474KA-T" H 2862 5726 50  0001 C CNN "SPURL"
-	1    2770 5580
+P 7360 1970
+F 0 "C15" H 7452 2016 50  0000 L CNN
+F 1 "100nF" H 7452 1925 50  0000 L CNN
+F 2 "Capacitor_SMD:C_0805_2012Metric_Pad1.15x1.40mm_HandSolder" H 7360 1970 50  0001 C CNN
+F 3 "https://www.mouser.com/datasheet/2/396/mlcc02_e-1307760.pdf" H 7360 1970 50  0001 C CNN
+F 4 "Multilayer Ceramic Capacitors MLCC - SMD/SMT 0603 6.3V 0.47uF 10% X7R" H 7452 2116 50  0001 C CNN "Description"
+F 5 "Taiyo Yuden" H 7360 1970 50  0001 C CNN "MFR"
+F 6 "JMK107B7474KA-T" H 7360 1970 50  0001 C CNN "MPN"
+F 7 "963-JMK107B7474KA-T" H 7452 2116 50  0001 C CNN "SPN"
+F 8 "Mouser" H 7360 1970 50  0001 C CNN "SPR"
+F 9 "https://www.mouser.com/ProductDetail/963-JMK107B7474KA-T" H 7452 2116 50  0001 C CNN "SPURL"
+	1    7360 1970
 	1    0    0    -1
 $EndComp
@@
 L Device:C_Small C16
 U 1 1 5F1175EF
-P 3150 5580
-F 0 "C16" H 3242 5626 50  0000 L CNN
-F 1 "100nF" H 3242 5535 50  0000 L CNN
-F 2 "Capacitor_SMD:C_0805_2012Metric_Pad1.15x1.40mm_HandSolder" H 3150 5580 50  0001 C CNN
-F 3 "https://www.mouser.com/datasheet/2/396/mlcc02_e-1307760.pdf" H 3150 5580 50  0001 C CNN
-F 4 "Multilayer Ceramic Capacitors MLCC - SMD/SMT 0603 6.3V 0.47uF 10% X7R" H 3242 5726 50  0001 C CNN "Description"
-F 5 "Taiyo Yuden" H 3150 5580 50  0001 C CNN "MFR"
-F 6 "JMK107B7474KA-T" H 3150 5580 50  0001 C CNN "MPN"
-F 7 "963-JMK107B7474KA-T" H 3242 5726 50  0001 C CNN "SPN"
-F 8 "Mouser" H 3150 5580 50  0001 C CNN "SPR"
-F 9 "https://www.mouser.com/ProductDetail/963-JMK107B7474KA-T" H 3242 5726 50  0001 C CNN "SPURL"
-	1    3150 5580
-	1    0    0    -1
-$EndComp
-Wire Wire Line
-	2770 5680 2960 5680
-Wire Wire Line
-	2770 5480 2960 5480
-Wire Wire Line
-	2960 5765 2960 5680
-Wire Wire Line
-	2960 5680 3150 5680
-Wire Wire Line
-	2960 5480 2960 5380
-Wire Wire Line
-	2960 5480 3150 5480
-Connection ~ 2960 5680
-Connection ~ 2960 5480
+P 7740 1970
+F 0 "C16" H 7832 2016 50  0000 L CNN
+F 1 "100nF" H 7832 1925 50  0000 L CNN
+F 2 "Capacitor_SMD:C_0805_2012Metric_Pad1.15x1.40mm_HandSolder" H 7740 1970 50  0001 C CNN
+F 3 "https://www.mouser.com/datasheet/2/396/mlcc02_e-1307760.pdf" H 7740 1970 50  0001 C CNN
+F 4 "Multilayer Ceramic Capacitors MLCC - SMD/SMT 0603 6.3V 0.47uF 10% X7R" H 7832 2116 50  0001 C CNN "Description"
+F 5 "Taiyo Yuden" H 7740 1970 50  0001 C CNN "MFR"
+F 6 "JMK107B7474KA-T" H 7740 1970 50  0001 C CNN "MPN"
+F 7 "963-JMK107B7474KA-T" H 7832 2116 50  0001 C CNN "SPN"
+F 8 "Mouser" H 7740 1970 50  0001 C CNN "SPR"
+F 9 "https://www.mouser.com/ProductDetail/963-JMK107B7474KA-T" H 7832 2116 50  0001 C CNN "SPURL"
+	1    7740 1970
+	1    0    0    -1
+$EndComp
+Wire Wire Line
+	7360 2070 7550 2070
+Wire Wire Line
+	7360 1870 7550 1870
+Wire Wire Line
+	7550 2155 7550 2070
+Wire Wire Line
+	7550 2070 7740 2070
+Wire Wire Line
+	7550 1870 7550 1770
+Wire Wire Line
+	7550 1870 7740 1870
+Connection ~ 7550 2070
+Connection ~ 7550 1870
 $Comp
 L power:+3V3 #PWR0120
 U 1 1 5F117603
-P 2960 5380
-F 0 "#PWR0120" H 2960 5230 50  0001 C CNN
-F 1 "+3V3" V 2975 5508 50  0000 L CNN
-F 2 "" H 2960 5380 50  0001 C CNN
-F 3 "" H 2960 5380 50  0001 C CNN
-	1    2960 5380
+P 7550 1770
+F 0 "#PWR0120" H 7550 1620 50  0001 C CNN
+F 1 "+3V3" V 7565 1898 50  0000 L CNN
+F 2 "" H 7550 1770 50  0001 C CNN
+F 3 "" H 7550 1770 50  0001 C CNN
+	1    7550 1770
 	1    0    0    -1
 $EndComp
@@
 L power:+5V #PWR0121
 U 1 1 5F1193D2
-P 2960 5765
-F 0 "#PWR0121" H 2960 5615 50  0001 C CNN
-F 1 "+5V" H 2975 5938 50  0000 C CNN
-F 2 "" H 2960 5765 50  0001 C CNN
-F 3 "" H 2960 5765 50  0001 C CNN
-	1    2960 5765
+P 7550 2155
+F 0 "#PWR0121" H 7550 2005 50  0001 C CNN
+F 1 "+5V" H 7565 2328 50  0000 C CNN
+F 2 "" H 7550 2155 50  0001 C CNN
+F 3 "" H 7550 2155 50  0001 C CNN
+	1    7550 2155
 	-1   0    0    1
 $EndComp
@@
 Wire Wire Line
 	3695 2160 3695 2205
+$Comp
+L 74xx:74HC3G04DP,125 U10
+U 1 1 5DABFD76
+P 8305 3325
+F 0 "U10" H 8485 3720 50  0000 C CNN
+F 1 "74HC3G04DP,125" H 8920 3720 50  0000 C CNN
+F 2 "Package_SO:TSSOP-8_3x3mm_P0.65mm" H 8305 3625 50  0001 C CNN
+F 3 "https://www.mouser.com/datasheet/2/916/74HC_HCT3G04-1319126.pdf" H 8305 3375 50  0001 C CNN
+	1    8305 3325
+	1    0    0    -1
+$EndComp
+$Comp
+L 74xx:74HC3G04DP,125 U10
+U 2 1 5DAC61A5
+P 8305 3525
+F 0 "U10" H 8485 4030 50  0000 C CNN
+F 1 "74HC3G04DP,125" H 8920 4030 50  0000 C CNN
+F 2 "Package_SO:TSSOP-8_3x3mm_P0.65mm" H 8305 3825 50  0001 C CNN
+F 3 "https://www.mouser.com/datasheet/2/916/74HC_HCT3G04-1319126.pdf" H 8305 3575 50  0001 C CNN
+	2    8305 3525
+	1    0    0    -1
+$EndComp
+$Comp
+L 74xx:74HC3G04DP,125 U10
+U 3 1 5DAC75F6
+P 8305 3725
+F 0 "U10" H 8490 4340 50  0000 C CNN
+F 1 "74HC3G04DP,125" H 8920 4345 50  0000 C CNN
+F 2 "Package_SO:TSSOP-8_3x3mm_P0.65mm" H 8305 4025 50  0001 C CNN
+F 3 "https://www.mouser.com/datasheet/2/916/74HC_HCT3G04-1319126.pdf" H 8305 3775 50  0001 C CNN
+	3    8305 3725
+	1    0    0    -1
+$EndComp
+$Comp
+L 74xx:74HC3G04DP,125 U10
+U 4 1 5DAC970E
+P 9490 2350
+F 0 "U10" H 9568 2371 50  0000 L CNN
+F 1 "74HC3G04DP,125" H 9568 2280 50  0000 L CNN
+F 2 "Package_SO:TSSOP-8_3x3mm_P0.65mm" H 9490 2650 50  0001 C CNN
+F 3 "https://www.mouser.com/datasheet/2/916/74HC_HCT3G04-1319126.pdf" H 9490 2400 50  0001 C CNN
+	4    9490 2350
+	1    0    0    -1
+$EndComp
 $EndSCHEMATC
