File: clocks.sch (KiCad schematic (older format))
At the start: 15 parts, among them J2 UPDI TTL, U10 74HC3G04DP,125, U11 MIC5356-SGYMME, U2 Si5351A-B-GT, U5 ATtiny1614-SS, Y1 25MHZ 8PF

Commit message: cleanup
Parts:
- removed C1, C2: 0.47uF, Capacitor_SMD:C_0603_1608Metric_Pad1.05x0.95mm_HandSolder, symbol Device:C_Small
- removed U10: 74HC3G04DP,125, Package_SO:TSSOP-8_3x3mm_P0.65mm, symbol 74xx:74HC3G04DP,125
- removed U11: MIC5356-SGYMME, Package_SO:MSOP-8-1EP_3x3mm_P0.65mm_EP2.5x3mm_Mask1.73x2.36mm_ThermalVias, symbol Regulator_Linear:MIC5356-SGYMME
- removed U2: Si5351A-B-GT, Package_SO:MSOP-10_3x3mm_P0.5mm, symbol Oscillator:Si5351A-B-GT
- added C15, C16: 0.47uF, Capacitor_SMD:C_0603_1608Metric_Pad1.05x0.95mm_HandSolder, symbol Device:C_Small
- added U10: 74HC04, symbol 74xx:74HC04
- added U2: TPS7A0533PDBVR, Package_TO_SOT_SMD:SOT-23-5, symbol Regulator_Linear:TPS7A0533PDBVR
- added U5: Si5351A-B-GT, Package_SO:MSOP-10_3x3mm_P0.5mm, symbol Oscillator:Si5351A-B-GT
- renumbered C15 to C1, C16 to C2, C4 to C3, C3 to C4, U5 to U11
Connections:
- wire segments 53 -> 58
Other:
- moved on the sheet: C3, C4

Commit message: added display, config switch
Parts:
- added U13: AS1115-BSST, Package_SO:QSOP-24_3.9x8.7mm_P0.635mm, symbol Interface_Expansion:AS1115-BSST
- added U14: ACDA02-41SGWA-F01, Display:ACDA02-41SGWA-F01, symbol Display_Character:ACDA02-41SGWA-F01
Connections:
- net labels added: D0, D1, D2, D3, D4, D5, D6, D7, D_ENA, SCL, SDA
- wire segments 58 -> 62
- no-connect marks 10 -> 1
Other:
- moved on the sheet: C1, C15, C16, C2, C3, C4, J2, R1, R2, R3, U10A, U10B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

Commit message: fixed NC pins
Parts:
- added R37: 9.53K, Resistor_SMD:R_0603_1608Metric_Pad1.05x0.95mm_HandSolder, symbol Device:R_Small
- U14: symbol Display_Character:ACDA02-41SGWA-F01 -> sbc_z80-rescue:ACDA02-41SGWA-F01-Display_Character
- U2: symbol Regulator_Linear:TPS7A0533PDBVR -> sbc_z80-rescue:TPS7A0533PDBVR-Regulator_Linear
Connections:
- net labels added: A, B, C, D, DIG0, DIG1, DP, E, F, G, IRQ
- net labels removed: D_ENA
- wire segments 62 -> 102
- no-connect marks 1 -> 9
Other:
- moved on the sheet: C15, C16, J2, R3, U11

Commit message: code for max7000 glue logic
Parts:
- C1, C15, C16, C2, C3, C4: symbol Device:C_Small -> sbc_z80-rescue:C_Small-Device
- J2: symbol Connector_Generic:Conn_01x03 -> sbc_z80-rescue:Conn_01x03-Connector_Generic
- R1, R2, R3, R37: symbol Device:R_Small -> sbc_z80-rescue:R_Small-Device
- U10: symbol 74xx:74HC04 -> sbc_z80-rescue:74HC04-74xx
- U11: symbol MCU_Microchip_ATtiny:ATtiny1614-SS -> sbc_z80-rescue:ATtiny1614-SS-MCU_Microchip_ATtiny
- U13: symbol Interface_Expansion:AS1115-BSST -> sbc_z80-rescue:AS1115-BSST-Interface_Expansion
- U5: symbol Oscillator:Si5351A-B-GT -> sbc_z80-rescue:Si5351A-B-GT-Oscillator
- Y1: symbol Device:Crystal_Small -> sbc_z80-rescue:Crystal_Small-Device
Changed lines of the file:
@@
 $EndDescr
 $Comp
-L Oscillator:Si5351A-B-GT U?
+L sbc_z80-rescue:Si5351A-B-GT-Oscillator U?
 U 1 1 5D255C0A
 P 8080 1505
@@
 $EndComp
 $Comp
-L Device:Crystal_Small Y1
+L sbc_z80-rescue:Crystal_Small-Device Y1
 U 1 1 5D255C0B
 P 7050 1305
@@
 $EndComp
 $Comp
-L power:GND #PWR?
+L sbc_z80-rescue:GND-power #PWR?
 U 1 1 5D255C0C
 P 8080 2005
@@
 $EndComp
 $Comp
-L Device:C_Small C15
+L sbc_z80-rescue:C_Small-Device C15
 U 1 1 5D255C0D
 P 3810 2495
@@
 $EndComp
 $Comp
-L Device:C_Small C16
+L sbc_z80-rescue:C_Small-Device C16
 U 1 1 5D255C0E
 P 4190 2495
@@
 $EndComp
 $Comp
-L power:GND #PWR?
+L sbc_z80-rescue:GND-power #PWR?
 U 1 1 5D00E3D9
 P 4000 2635
@@
 $EndComp
 $Comp
-L Device:R_Small R1
+L sbc_z80-rescue:R_Small-Device R1
 U 1 1 5D0168D6
 P 6530 1325
@@
 $EndComp
 $Comp
-L Device:R_Small R2
+L sbc_z80-rescue:R_Small-Device R2
 U 1 1 5D017809
 P 6730 1325
@@
 Connection ~ 6630 1165
 $Comp
-L MCU_Microchip_ATtiny:ATtiny1614-SS U11
+L sbc_z80-rescue:ATtiny1614-SS-MCU_Microchip_ATtiny U11
 U 1 1 5D018E69
 P 5395 2105
@@
 	5395 1405 5395 1305
 $Comp
-L power:GND #PWR?
+L sbc_z80-rescue:GND-power #PWR?
 U 1 1 5D01D4B0
 P 5395 2805
@@
 $EndComp
 $Comp
-L Connector_Generic:Conn_01x03 J?
+L sbc_z80-rescue:Conn_01x03-Connector_Generic J?
 U 1 1 5D03DC78
 P 3490 1705
@@
 TX
 $Comp
-L Device:R_Small R3
+L sbc_z80-rescue:R_Small-Device R3
 U 1 1 5D041A40
 P 4355 1705
@@
 CLK_7_3728_Mhz
 $Comp
-L power:GND #PWR?
+L sbc_z80-rescue:GND-power #PWR?
 U 1 1 5D4AC760
 P 9095 3435
@@
 $EndComp
 $Comp
-L Device:C_Small C4
+L sbc_z80-rescue:C_Small-Device C4
 U 1 1 5D1521F5
 P 1265 1045
@@
 $EndComp
 $Comp
-L Device:C_Small C3
+L sbc_z80-rescue:C_Small-Device C3
 U 1 1 5D152201
 P 2570 1040
@@
 $EndComp
 $Comp
-L power:GND #PWR?
+L sbc_z80-rescue:GND-power #PWR?
 U 1 1 5D15A1D6
 P 1980 1390
@@
 Connection ~ 2570 945
 $Comp
-L power:+3V3 #PWR03
+L sbc_z80-rescue:+3V3-power #PWR03
 U 1 1 5EFB1AF8
 P 2875 945
@@
 $EndComp
 $Comp
-L power:+3V3 #PWR039
+L sbc_z80-rescue:+3V3-power #PWR039
 U 1 1 5EFB3E73
 P 4000 2295
@@
 $EndComp
 $Comp
-L power:+3V3 #PWR036
+L sbc_z80-rescue:+3V3-power #PWR036
 U 1 1 5EFB591E
 P 5395 1305
@@
 $EndComp
 $Comp
-L power:+3V3 #PWR034
+L sbc_z80-rescue:+3V3-power #PWR034
 U 1 1 5EFB7DBF
 P 6630 1105
@@
 $EndComp
 $Comp
-L power:+3V3 #PWR033
+L sbc_z80-rescue:+3V3-power #PWR033
 U 1 1 5EFB9342
 P 8080 905
@@
 $EndComp
 $Comp
-L power:+5V #PWR040
+L sbc_z80-rescue:+5V-power #PWR040
 U 1 1 5EFBA650
 P 9095 2435
@@
 	3895 1370 3895 1420
 $Comp
-L power:GND #PWR?
+L sbc_z80-rescue:GND-power #PWR?
 U 1 1 5EFBCFCB
 P 3895 1420
@@
 $EndComp
 $Comp
-L power:PWR_FLAG #FLG02
+L sbc_z80-rescue:PWR_FLAG-power #FLG02
 U 1 1 5EFC0EF3
 P 2785 945
@@
 	2785 945  2875 945
 $Comp
-L power:PWR_FLAG #FLG01
+L sbc_z80-rescue:PWR_FLAG-power #FLG01
 U 1 1 5EFC1C86
 P 1120 945
@@
 Connection ~ 1120 945
 $Comp
-L Device:C_Small C1
+L sbc_z80-rescue:C_Small-Device C1
 U 1 1 5F1175E3
 P 900 2280
@@
 $EndComp
 $Comp
-L Device:C_Small C2
+L sbc_z80-rescue:C_Small-Device C2
 U 1 1 5F1175EF
 P 1280 2280
@@
 Connection ~ 1090 2180
 $Comp
-L power:+3V3 #PWR01
+L sbc_z80-rescue:+3V3-power #PWR01
 U 1 1 5F117603
 P 1090 2080
@@
 $EndComp
 $Comp
-L power:+5V #PWR07
+L sbc_z80-rescue:+5V-power #PWR07
 U 1 1 5F1193D2
 P 1090 2465
@@
 $EndComp
 $Comp
-L power:+5V #PWR02
+L sbc_z80-rescue:+5V-power #PWR02
 U 1 1 5F57C70A
 P 715 945
@@
 	1475 1045 1475 945
 $Comp
-L power:GND #PWR?
+L sbc_z80-rescue:GND-power #PWR?
 U 1 1 5E77B1C8
 P 2570 1185
@@
 	2570 1140 2570 1185
 $Comp
-L power:GND #PWR?
+L sbc_z80-rescue:GND-power #PWR?
 U 1 1 5E77C6D4
 P 1265 1190
@@
 	8845 1305 8845 1080
 $Comp
-L 74xx:74HC04 U10
+L sbc_z80-rescue:74HC04-74xx U10
 U 1 1 5D29C9BF
 P 9145 1080
@@
 $EndComp
 $Comp
-L 74xx:74HC04 U10
+L sbc_z80-rescue:74HC04-74xx U10
 U 2 1 5D2A53E5
 P 9140 1505
@@
 $EndComp
 $Comp
-L 74xx:74HC04 U10
+L sbc_z80-rescue:74HC04-74xx U10
 U 3 1 5D2A9AD2
 P 9140 1925
@@
 $EndComp
 $Comp
-L 74xx:74HC04 U10
+L sbc_z80-rescue:74HC04-74xx U10
 U 7 1 5D2AB645
 P 9095 2935
@@
 $EndComp
 $Comp
-L 74xx:74HC04 U10
+L sbc_z80-rescue:74HC04-74xx U10
 U 6 1 5D2DEE4B
 P 7400 3175
@@
 	7010 3175 7010 3235
 $Comp
-L power:GND #PWR?
+L sbc_z80-rescue:GND-power #PWR?
 U 1 1 5D2E3B91
 P 7010 3235
@@
 IRQ
 $Comp
-L Interface_Expansion:AS1115-BSST U?
+L sbc_z80-rescue:AS1115-BSST-Interface_Expansion U?
 U 1 1 5F4897F0
 P 2635 4585
@@
 SDA
 $Comp
-L power:GND #PWR?
+L sbc_z80-rescue:GND-power #PWR?
 U 1 1 5D361F7F
 P 2635 5785
@@
 	2635 3385 2635 3330
 $Comp
-L power:+3V3 #PWR047
+L sbc_z80-rescue:+3V3-power #PWR047
 U 1 1 5D369131
 P 2635 3285
@@
 $EndComp
 $Comp
-L Device:R_Small R37
+L sbc_z80-rescue:R_Small-Device R37
 U 1 1 5D374E92
 P 1795 3605
