File: sbc_z80.sch (KiCad schematic (older format))
At the start: 61 parts, among them J1 RC80 Bus, J3 PIO Header, J4 Conn_01x06, J5 Conn_01x06, J6 CTC Header, J7 AVR-JTAG-10, SW1 SW_Push, SW2 SW_DIP_x06, U1 CPU - Z84C0010AEG, U10 74HC04, U12 MIC811LUY, U3 SRAM - IS62C5128BL-45TLI, U4 GLS29EE010, U6 SIO/3 - Z84C4310AEG, U7 CPLD - EPM7032STC44, U8 CTC - Z84C3010AEG, U9 PIO - Z84C2010AEG

Commit message: fixed NC pins
Parts:
- U1: symbol sbc_z80-rescue:Z84C0010AEG-zilog -> sbc_z80-rescue:Z84C0010AEG
- U6: symbol sbc_z80-rescue:Z84C4310AEG-zilog -> sbc_z80-rescue:Z84C4310AEG
- U8: symbol sbc_z80-rescue:Z84C3010AEG-zilog -> sbc_z80-rescue:Z84C3010AEG
- U9: value PIO - Z84C2010AEG -> Z84C2010AEG; symbol sbc_z80-rescue:Z84C2010AEG-zilog -> sbc_z80-rescue:Z84C2010AEG
Connections:
- no-connect marks 18 -> 19
Other:
- moved on the sheet: J3, J6, R25, R26, R27, R28, R31, R32, R33, R34, R35, R36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

Commit message: code for max7000 glue logic
Parts:
- C10, C11, C12, C13, C14, C5, C6, C7, C8, C9: symbol Device:C_Small -> sbc_z80-rescue:C_Small-Device
- D1: symbol Device:LED_Dual_ACAC -> sbc_z80-rescue:LED_Dual_ACAC-Device
- J1: symbol Connector_Generic:Conn_02x40_Top_Bottom -> sbc_z80-rescue:Conn_02x40_Top_Bottom-Connector_Generic
- J3: symbol Connector_Generic:Conn_02x13_Odd_Even -> sbc_z80-rescue:Conn_02x13_Odd_Even-Connector_Generic
- J4, J5: symbol Connector_Generic:Conn_01x06 -> sbc_z80-rescue:Conn_01x06-Connector_Generic
- J6: symbol Connector_Generic:Conn_01x10 -> sbc_z80-rescue:Conn_01x10-Connector_Generic
- J7: symbol Connector:AVR-JTAG-10 -> sbc_z80-rescue:AVR-JTAG-10-Connector
- R10, R11, R12, R13, R14, R15, R16, R17, R18, R19, R20, R21, R22, R23, R24, R25, R26, R27, R28, R29, R30, R31, R32, R33, R34, R35, R36, R4, R5, R6, R7, R8, R9: symbol Device:R_Small -> sbc_z80-rescue:R_Small-Device
- SW1: symbol Switch:SW_Push -> sbc_z80-rescue:SW_Push-Switch
- SW2: symbol Switch:SW_DIP_x06 -> sbc_z80-rescue:SW_DIP_x06-Switch
- U10: symbol 74xx:74HC04 -> sbc_z80-rescue:74HC04-74xx
- U12: symbol Power_Supervisor:MIC811LUY -> sbc_z80-rescue:MIC811LUY-Power_Supervisor
Connections:
- net TDO: now also U7.32 (B20/TDO); no longer U7.31 (B21)
- net ~CTC: now also U7.31 (B21); no longer U7.32 (B20/TDO)
